Commit message: ur5_arm urdf

File: ur5_pick_place/gripper_description/urdf/gripper.gazebo.xacro (robot description, xacro)
@@ -1,5 +1,5 @@
 <?xml version="1.0"?>
-<robot>
-    <xacro:macro name="gripper_gazebo" params="prefix">
+<robot xmlns:xacro="http://wiki.ros.org/xacro">
+  <xacro:macro name="gripper_gazebo" params="prefix">
       <gazebo reference="${prefix}gripper_link">
         <material>Gazebo/Grey</material>

File: ur5_pick_place/gripper_description/urdf/gripper.urdf.xacro (robot description, xacro)
@@ -1,4 +1,6 @@
 <?xml version="1.0"?>
 <robot xmlns:xacro="http://wiki.ros.org/xacro" name="gripper">
+    <!--XACRO ARGUMENTS-->
+    <xacro:arg name="prefix" default=""/>
     <!--XACRO INCLUDES-->
     <xacro:include filename="$(find gripper_description)/urdf/gripper.gazebo.xacro" />
@@ -68,5 +70,5 @@
             <child link="right_gripper_finger_link" />
             <axis xyz="0 1 0" />
-            <limit effort="100" lower="-0.01" upper="0.06" velocity="0.05" />
+            <limit effort="100" lower="-0.01" upper="0.03" velocity="0.05" />
             <dynamics damping="0.7" />
         </joint>
@@ -76,5 +78,5 @@
             <child link="left_gripper_finger_link" />
             <axis xyz="0 -1 0" />
-            <limit effort="100" lower="-0.01" upper="0.06" velocity="0.05" />
+            <limit effort="100" lower="-0.01" upper="0.03" velocity="0.05" />
             <dynamics damping="0.7" />
         </joint>
@@ -83,4 +85,4 @@
     </xacro:macro>
     <!--GRIPPER URDF-->
-    <xacro:gripper prefix="${prefix}" />
+    <xacro:gripper prefix="$(arg prefix)"/>
 </robot>

Commit message: improved URDF

File: ur5_pick_place/gripper_description/urdf/gripper.gazebo.xacro (robot description, xacro)
@@ -2,9 +2,4 @@
 <robot xmlns:xacro="http://wiki.ros.org/xacro">
   <xacro:macro name="gripper_gazebo" params="prefix">
-      <gazebo>
-        <plugin name="gazebo_ros_control" filename="libgazebo_ros_control.so">
-          <robotNamespace>${prefix}gripper</robotNamespace>
-        </plugin>
-      </gazebo>
       <gazebo reference="${prefix}gripper_link">
         <material>Gazebo/Grey</material>
@@ -26,22 +21,4 @@
         <mu2>30.0</mu2>
       </gazebo>
-      <!-- grasp plugin -->
-       <gazebo>
-         <plugin name="gazebo_grasp_fix" filename="libgazebo_grasp_fix.so">
-           <arm>
-             <arm_name>ur5_arm</arm_name>
-             <palm_link>ee_link</palm_link>
-             <gripper_link>right_gripper_finger_link</gripper_link>
-             <gripper_link>left_gripper_finger_link</gripper_link>
-           </arm>
-           <forces_angle_tolerance>100</forces_angle_tolerance>
-           <update_rate>4</update_rate>
-           <grip_count_threshold>4</grip_count_threshold>
-           <max_grip_count>8</max_grip_count>
-           <release_tolerance>0.001</release_tolerance>
-           <disable_collisions_on_attach>false</disable_collisions_on_attach>
-           <contact_topic>__default_topic__</contact_topic>
-         </plugin>
-       </gazebo>
     </xacro:macro>
 </robot>

File: ur5_pick_place/gripper_description/urdf/gripper.urdf.xacro (robot description, xacro)
@@ -2,5 +2,5 @@
 <robot xmlns:xacro="http://wiki.ros.org/xacro" name="gripper">
     <!--XACRO ARGUMENTS-->
-    <xacro:arg name="prefix" default=""/>
+    <!--<xacro:arg name="prefix" default=""/>-->
     <!--XACRO INCLUDES-->
     <xacro:include filename="$(find gripper_description)/urdf/gripper.gazebo.xacro" />
@@ -81,8 +81,9 @@
             <dynamics damping="0.7" />
         </joint>
+        <!--XACRO MACRO-->
         <xacro:gripper_transmission prefix="${prefix}" />
         <xacro:gripper_gazebo prefix="${prefix}" />
     </xacro:macro>
     <!--GRIPPER URDF-->
-    <xacro:gripper prefix="$(arg prefix)"/>
+    <!--<xacro:gripper prefix="$(arg prefix)"/>-->
 </robot>

File: ur5_pick_place/ur5_arm_description/urdf/ur5_arm.urdf.xacro (robot description, xacro)
@@ -1,7 +1,18 @@
 <?xml version="1.0"?>
 <robot xmlns:xacro="http://wiki.ros.org/xacro" name="ur5_arm">
+    <!--XACRO ARGUMENTS-->
+    <xacro:arg name="prefix" default=""/>
+    <xacro:arg name="joint_limited" default="false"/>
+    <xacro:arg name="transmission_hw_interface" default="hardware_interface/PositionJointInterface"/>
     <!--XACRO INCLUDES-->
     <xacro:include filename="$(find gripper_description)/urdf/gripper.urdf.xacro" />
-    <xacro:include filename="$(find ur_description)/urdf/ur5_robot.urdf.xacro" />
+    <xacro:include filename="$(find ur_description)/urdf/ur5.urdf.xacro" />
+    <xacro:include filename="$(find ur5_arm_description)/urdf/gazebo_plugins.urdf.xacro" />
+    <!--GRIPPER MACRO-->
+    <xacro:gripper prefix="$(arg prefix)"/>
+    <!--UR5 MACRO-->
+    <xacro:ur5_robot prefix="$(arg prefix)" joint_limited="$(arg joint_limited)"
+    transmission_hw_interface="$(arg transmission_hw_interface)"
+    />
     <!--ROBOT LAST LINK TO GRIPPER BASE LINK-->
     <joint name="gripper_joint" type="fixed">
@@ -11,3 +22,9 @@
         <axis xyz="0 1 0" />
     </joint>
+    <!--GAZEBO FIX URDF TO WORLD-->
+    <link name="world" />
+    <joint name="world_joint" type="fixed">
+        <parent link="world" />
+        <child link = "base_link" />
+    </joint>
 </robot>
